Commit message: Publishing cone detections in sensors' frame
- added camera_center frame for camera cone detections representation

File: fssim_description/urdf/vehicle/sensors.xacro (robot description, xacro)
@@ -25,4 +25,16 @@
     </xacro:macro>
     <xacro:macro name="camera_pipeline">
+        <!-- Sensor links and fixed joints -->
+        <link name="camera_center_link">
+            <inertial>
+                <mass value="1"/>
+                <inertia ixx="0.001" ixy="0.0" ixz="0.0" iyy="0.001" iyz="0.0" izz="0.001"/>
+            </inertial>
+        </link>
+        <joint name="camera_center_joint" type="fixed">
+            <parent link="chassis"/>
+            <child link="camera_center_link"/>
+            <origin xyz="${sensors['camera']['pos']['x']} 0.0 0.15" rpy="0 0 0"/>
+        </joint>
         <gazebo>
             <plugin name="camera_pipeline" filename="libgazebo_cone_sensor.so">
